File: biastee/LNA-BiasT.kicad_pcb (KiCad board)
At the start: 2 copper layers, 50 x 29 mm, 15 parts, among them CON1 DC, P1 ANT, P2 RX, U1 LM317AEMP

Commit message: added more decoupling capacitors
Parts:
- added C6: 10nF, Capacitors_SMD:C_0603_HandSoldering, F.Cu at (140.0, 77.0)
- added C7: 1nF, Capacitors_SMD:C_0603_HandSoldering, F.Cu at (140.0, 78.6)
- added C8: 100pF, Capacitors_SMD:C_0603_HandSoldering, F.Cu at (140.0, 80.2)
Routing:
- net /REGOUT: track 33.5 -> 42.3 mm
- net GND: track 557.7 -> 550.5 mm, vias 312 -> 309
