File: miniwhip/miniwhip.kicad_pcb (KiCad board)
At the start: 2 copper layers, 80 x 32 mm, 17 parts, among them P1 MINIWHIP, P2 BNC, Q1 MMBF5485, Q2 BFR92

Commit message: changed silksreen slightly
Other:
- board text added: "PA0RDT MiniWhip Rev. A 2015 g4lvanix"
- board text removed: "PA0RDT MiniWhip Rev. A 2015 devthrash"
Changed lines of the file:
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@@
-(kicad_pcb (version 4) (host pcbnew "(2015-05-21 BZR 5674)-product")
+(kicad_pcb (version 4) (host pcbnew "(2015-07-09 BZR 5919)-product")
   (general
     (links 26)
@@
     )
   )
-  (gr_text "PA0RDT MiniWhip Rev. A\n2015 devthrash\n" (at 134 91) (layer F.Mask)
+  (gr_text "PA0RDT MiniWhip Rev. A\n2015 g4lvanix" (at 134 91) (layer F.Mask)
     (effects (font (size 1.5 1.5) (thickness 0.3)))
   )
